File: RFID_BREAKOUT/RFID_BREAKOUT.kicad_pcb (KiCad board)
At the start: 2 copper layers, 140 x 45 mm, 12 parts, among them J1 Conn_02x08_Odd_Even, J10 Conn_02x08_Odd_Even, J11 Conn_02x08_Odd_Even, J13 Conn_02x05_Odd_Even, J2 Conn_01x20_Pin, J3 Conn_02x08_Odd_Even, J4 Conn_02x08_Odd_Even, J5 Conn_02x08_Odd_Even, J6 Conn_02x08_Odd_Even, J7 Conn_02x08_Odd_Even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

Commit message: 15oct
Parts:
- moved J2 5.00 mm to (195.0, 77.5)
Routing:
- net /RST1: track 162.4 -> 174.7 mm
- net /RST2: track 147.3 -> 159.1 mm
- net /RST3: track 132.3 -> 143.5 mm
- net /RST4: track 117.3 -> 127.9 mm
- net /RST5: track 102.3 -> 111.6 mm
- net /RST6: track 87.2 -> 96.0 mm
- net /RST8: track 57.0 -> 64.1 mm
- net /SDA2: track 107.4 -> 114.1 mm
- net /RST7: track 73.2 -> 79.6 mm
- net /SDA1: track 117.2 -> 123.5 mm
- net /RST9: track 41.9 -> 47.7 mm
- net /RST10: track 26.5 -> 31.7 mm
- net /SDA3: track 99.0 -> 103.7 mm
- net /SDA10: track 36.8 -> 33.4 mm
- net /SDA9: track 46.9 -> 43.7 mm
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Other:
- board size 140 x 45 mm -> 150 x 55 mm
